File: kicad/divider.sch (KiCad schematic (older format))
At the start: 25 parts, among them J1 CLK, J10 CLKTN GND, J2 RESET, J3 RESET GND, Q1 2N3904, Q2 2N3904, Q3 2N3904, Q4 2N3904, U1 4024

Commit message: Use 6V. Add output diodes + output pin headers
Parts:
- C1: footprint Capacitor_SMD:C_01005_0402Metric -> Capacitor_SMD:C_0402_1005Metric
Changed lines of the file:
@@
 F 0 "C1" H 1718 7046 50  0000 L CNN
 F 1 "1u" H 1718 6955 50  0000 L CNN
-F 2 "Capacitor_SMD:C_01005_0402Metric" H 1638 6850 50  0001 C CNN
+F 2 "Capacitor_SMD:C_0402_1005Metric" H 1638 6850 50  0001 C CNN
 F 3 "https://datasheet.lcsc.com/szlcsc/Samsung-Electro-Mechanics-CL05A105KA5NQNC_C52923.pdf" H 1600 7000 50  0001 C CNN
 F 4 "C52923" H 1600 7000 50  0001 C CNN "LCSC"
